Commit message: Creation of agrosim package

File: src/warthog/warthog_description/urdf/warthog.urdf.xacro (robot description, xacro)
@@ -349,5 +349,5 @@
     </link>
     <joint name="joint_sensor_laser" type="fixed">
-    <origin xyz="0.3 0 0.2" rpy="0 0 0"/>
+    <origin xyz="0.3 0 0.2" rpy="0 -0.2 0"/>
     <parent link="base_link"/>
     <child link="base_laser_link"/>
@@ -405,4 +405,46 @@
     </sensor>
   </gazebo>
+<gazebo reference="base_laser_link">
+  <sensor name="base_laser_link_camera" type="depth">
+    <update_rate>20</update_rate>
+    <camera>
+      <horizontal_fov>1.047198</horizontal_fov>
+      <image>
+        <width>640</width>
+        <height>480</height>
+        <format>R8G8B8</format>
+      </image>
+      <clip>
+        <near>0.05</near>
+        <far>9</far>
+      </clip>
+    </camera>
+    <plugin name="base_laser_link_controller" filename="libgazebo_ros_openni_kinect.so">
+      <baseline>0.2</baseline>
+      <alwaysOn>true</alwaysOn>
+      <updateRate>1.0</updateRate>
+      <namespace></namespace>
+      <cameraName>camera</cameraName>
+      <!-- <imageTopicName>/Camera/color/image_raw</imageTopicName>
+      <cameraInfoTopicName>/Camera/color/camera_info</cameraInfoTopicName>
+      <depthImageTopicName>/Camera/depth/image_raw</depthImageTopicName>
+      <depthImageInfoTopicName>/Camera/depth/camera_info</depthImageInfoTopicName>
+      <pointCloudTopicName>/Camera/depth/points</pointCloudTopicName> -->
+      <frameName>base_laser_link</frameName>
+      <pointCloudCutoff>0.5</pointCloudCutoff>
+      <pointCloudCutoffMax>3.0</pointCloudCutoffMax>
+      <distortionK1>0.00000001</distortionK1>
+      <distortionK2>0.00000001</distortionK2>
+      <distortionK3>0.00000001</distortionK3>
+      <distortionT1>0.00000001</distortionT1>
+      <distortionT2>0.00000001</distortionT2>
+      <CxPrime>0</CxPrime>
+      <Cx>0</Cx>
+      <Cy>0</Cy>
+      <focalLength>0</focalLength>
+      <hackBaseline>0</hackBaseline>
+    </plugin>
+  </sensor>
+</gazebo>
   <gazebo>
   <plugin name="ground_truth" filename="libgazebo_ros_p3d.so">
